File: pcb/ft2232h.sch (KiCad schematic (older format))
At the start: 39 parts, among them P1 CONN_01X16, P2 CONN_01X16, P3 CONN_01X02, SW1 SW_PUSH_SMALL, U1 AMS1117, U2 eeprom_93LC56B, U3 FT2232H, X1 micro_USB, Y1 12MHz

Commit message: Update ft2232h.sch
Parts:
- removed C1, C8: 100nF, symbol C_Small
- removed C12: 0.1uF, symbol C_Small
- removed C15, C16, C17, C18, C19, C20, C7, C?: 0.1uF/50V, Capacitors_SMD:C_0805, symbol C_Small
- removed C2, C5: 27pF, symbol C_Small
- removed C3, C4: 4.7uF, symbol CP
- removed FB2: FerriteB, symbol FerriteB
- removed P1, P2: CONN_01X16, symbol CONN_01X16
- removed P3: CONN_01X02, symbol CONN_01X02
- removed R3, R5: 10kOhm, symbol R_Small
- removed U2: eeprom_93LC56B, symbol eeprom_93LC56B
- removed Y1: 12MHz, symbol Crystal_Small
- added C1, C10, C13, C14, C15, C16, C17, C18, C19, C5, C6: 0.1uF/50V, Capacitor_SMD:C_0805_2012Metric_Pad1.15x1.40mm_HandSolder, symbol sjtag-rescue:C_Small
- added C2, C3: 4.7uF/10V, Capacitor_Tantalum_SMD:CP_EIA-3216-18_Kemet-A_Pad1.58x1.35mm_HandSolder, symbol sjtag-rescue:CP
- added FB2: FerriteB, footprints:FerriteBead, symbol symbols:FerriteB
- added J1, J2: PBD-6, Connector_PinSocket_2.54mm:PinSocket_2x03_P2.54mm_Vertical, symbol Connector_Generic:Conn_02x03_Odd_Even
- added J3, J4: PBD-2x10, Connector_PinSocket_2.54mm:PinSocket_2x10_P2.54mm_Vertical, symbol Connector_Generic:Conn_02x10_Odd_Even
- added R3, R5: 10kOhm, Resistor_SMD:R_0805_2012Metric_Pad1.15x1.40mm_HandSolder, symbol sjtag-rescue:R_Small
- added R7, R8: 10 Ohm, Resistor_SMD:R_0805_2012Metric_Pad1.15x1.40mm_HandSolder, symbol sjtag-rescue:R_Small
- added U2: eeprom_93C46, Package_SO:SOIC-8_3.9x4.9mm_P1.27mm, symbol symbols:eeprom_93C46
- added Y1: 12MHz, footprints:CSTCE_G15C, symbol symbols:Crystal_CSTCE_G15C
- C11: renamed from C13; footprint Capacitors_SMD:C_0805 -> Capacitor_SMD:C_0805_2012Metric_Pad1.15x1.40mm_HandSolder; symbol C_Small -> sjtag-rescue:C_Small
- C12: renamed from C14; footprint (none) -> Capacitor_SMD:C_0805_2012Metric_Pad1.15x1.40mm_HandSolder; symbol C_Small -> sjtag-rescue:C_Small; PN (none) -> GRM21BR60J335KA11L
- C4: renamed from C6; value 10uF/10V -> 4.7uF/10V; footprint Capacitors_Tantalum_SMD:TantalC_SizeA_EIA-3216_HandSoldering -> Capacitor_Tantalum_SMD:CP_EIA-3216-18_Kemet-A_Pad1.58x1.35mm_HandSolder; symbol CP -> sjtag-rescue:CP; PN TECAP10/10VA10 -> TECAP4.7/10VA10
- C7: renamed from C9; footprint Capacitors_SMD:C_0805 -> Capacitor_SMD:C_0805_2012Metric_Pad1.15x1.40mm_HandSolder; symbol C_Small -> sjtag-rescue:C_Small
- C8: renamed from C10; value 10uF/10V -> 4.7uF/10V; footprint Capacitors_Tantalum_SMD:TantalC_SizeA_EIA-3216_HandSoldering -> Capacitor_Tantalum_SMD:CP_EIA-3216-18_Kemet-A_Pad1.58x1.35mm_HandSolder; symbol CP -> sjtag-rescue:CP; PN TECAP10/10VA10 -> TECAP4.7/10VA10
- C9: renamed from C11; footprint Capacitors_SMD:C_0805 -> Capacitor_SMD:C_0805_2012Metric_Pad1.15x1.40mm_HandSolder; symbol C_Small -> sjtag-rescue:C_Small
- F1: footprint (none) -> footprints:MF-MSMF050; symbol F_Small -> sjtag-rescue:F_Small; PN (none) -> MF-MSMF050
- FB1: footprint (none) -> footprints:FerriteBead; symbol FerriteB -> symbols:FerriteB; PN (none) -> MMZ2012Y601BT000
- R1: footprint (none) -> Resistor_SMD:R_0805_2012Metric_Pad1.15x1.40mm_HandSolder; symbol R_Small -> sjtag-rescue:R_Small; PN (none) -> RC0805FR-071KL
- R2: footprint (none) -> Resistor_SMD:R_0805_2012Metric_Pad1.15x1.40mm_HandSolder; symbol R_Small -> sjtag-rescue:R_Small; PN (none) -> RC0805FR-0710KL
- R4: footprint (none) -> Resistor_SMD:R_0805_2012Metric_Pad1.15x1.40mm_HandSolder; symbol R_Small -> sjtag-rescue:R_Small; PN (none) -> RC0805FK-072KL
- R6: footprint (none) -> Resistor_SMD:R_0805_2012Metric_Pad1.15x1.40mm_HandSolder; symbol R_Small -> sjtag-rescue:R_Small; PN (none) -> RC0805FR-0712KL
- SW1: footprint (none) -> footprints:IT-1185AP; symbol SW_PUSH_SMALL -> sjtag-rescue:SW_PUSH_SMALL; PN (none) -> 1437566-3 (FSMSM); PN2 (none) -> IT-1185AP
- U1: footprint (none) -> Package_TO_SOT_SMD:SOT-223; symbol AMS1117 -> symbols:AMS1117; PN (none) -> AMS1117-3.3
- U3: footprint (none) -> Package_QFP:LQFP-64_10x10mm_P0.5mm; symbol FT2232H -> symbols:FT2232H; PN (none) -> FT2232HL-REEL
- X1: symbol micro_USB -> symbols:micro_USB
Connections:
- net labels added: 3.3V_out, 5V_out, DM_N, DP_P
- net labels removed: dm, dp
- wire segments 194 -> 264
