File: pcb/ft2232h.kicad_pcb (KiCad board)
At the start: 2 copper layers, 75 x 40 mm, 40 parts, among them J1 PBD-6, J2 PBD-6, J3 PBD-2x10, J4 PBD-2x10, SW1 SW_PUSH_SMALL, U1 AMS1117, U2 eeprom_93C46, U3 FT2232H, X1 micro_USB, Y1 12MHz

Commit message: redraw pcb
Parts:
- moved C1 39.3 mm to (90.6, 114.7), turned to 180 degrees
- moved R1 33.1 mm to (90.6, 109.8), turned to 0 degrees
- moved Reset 11.0 mm to (121.2, 102.0), turned to 270 degrees
- moved J4 9.00 mm to (98.0, 81.5)
- moved J3 9.00 mm to (98.0, 116.0)
- moved R6 5.52 mm to (80.7, 95.1), turned to 0 degrees
- moved R4 4.74 mm to (97.8, 87.4)
- moved R5 4.43 mm to (90.8, 87.4)
- moved R2 3.90 mm to (90.7, 92.9)
- moved R3 3.73 mm to (90.8, 90.5)
- moved C12 3.55 mm to (111.4, 92.8), turned to 0 degrees
- moved C15 3.20 mm to (100.4, 92.1), turned to 180 degrees
- moved U2 2.99 mm to (90.6, 89.3)
- moved C10 2.79 mm to (83.7, 90.1), turned to 90 degrees
- moved C6 2.68 mm to (85.2, 95.2)
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- renumbered SW1 to Reset
Routing:
- net /3.3V: track 254.9 -> 228.9 mm
- net /rst: track 63.3 -> 50.4 mm
- net /ACBUS7: track 33.1 -> 21.0 mm
- net /ACBUS5: track 27.9 -> 16.1 mm
- net /ACBUS6: track 30.5 -> 19.7 mm
- net /ACBUS4: track 26.0 -> 15.4 mm
- net /ACBUS3: track 24.0 -> 14.6 mm
- net /ADBUS4: track 27.4 -> 18.5 mm
- net /ADBUS7: track 32.7 -> 23.9 mm
- net /ADBUS5: track 29.2 -> 20.4 mm
- net /ADBUS1: track 22.2 -> 13.5 mm
- net /ADBUS2: track 24.2 -> 15.5 mm
- net /ADBUS6: track 31.0 -> 22.4 mm
- net /ADBUS3: track 26.0 -> 17.4 mm
- net /ACBUS2: track 21.6 -> 13.7 mm
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- added copper zone on F.Cu, net /3.3V
Other:
- board size 75 x 40 mm -> 63 x 40 mm
- board text added: "0"
- board text added: "1"
- board text added: "2"
- board text added: "3"
- board text added: "4"
- board text added: "5"
- board text added: "6"
- board text added: "7"

Commit message: plot GND, schematic to pdf
Parts:
- moved C1 5.06 mm to (89.9, 109.7)
- moved R1 2.88 mm to (89.9, 107.1)
Routing:
- net /rst: track 50.4 -> 47.3 mm
- net /3.3V: track 228.9 -> 230.9 mm
- net Earth: vias 0 -> 8
- added copper zone on B.Cu, net Earth
- added copper zone on F.Cu, net Earth
Other:
- rule via_min_size: 0.4 -> 1.4
- board text added: "3V3_out"
- board text added: "5V_out"
- board text added: "ACBUSx"
- board text added: "ADBUSx"
- board text added: "BCBUSx"
- board text added: "BDBUSx"
- board text added: "GND"
- board text added: "pwren"
- board text added: "suspend"
